File: matrix_display16_32/matrix_control_main/matrix_control_main.kicad_pcb (KiCad board)
At the start: 2 copper layers, 96.5 x 45.7 mm, 43 parts, among them J1 Conn_01x05_Male, J2 Conn_01x04_Male, P1 Connector_USB_C_Plug_USB2.0, P666 CON_1, Q1 SOT-23_SS8050_Y1, SW1 RST, SW2 Dowload, U1 ESP-12, U2 CH340E, U3 DS3231, U4 XC6228D332VR-G

Commit message: 修改matrix_display16_32 3D模型封装
Parts:
- removed P666 (x2): CON_1, NewLibCool:CON1
- D2: footprint lc_lib:0603_LED_S1 -> LED_SMD:LED_0603_1608Metric
- J1: footprint Connector_PinHeader_2.00mm:PinHeader_1x05_P2.00mm_Vertical -> Connector_PinSocket_2.00mm:PinSocket_1x05_P2.00mm_Vertical
- J2: footprint Connector_PinHeader_2.54mm:PinHeader_1x04_P2.54mm_Vertical -> matrix_control_main:Pin_1x04_P2.54mm_DHT11
- P1: footprint matrix_control_main:USB-Type-C -> WDebug_DAPLink:USB-Type-C
- SW1, SW2: footprint matrix_control_main:SWITCH_PUSH -> WDebug_DAPLink:SWITCH_PUSH
Routing:
- net Net-(D2-PadK): track 2.65 -> 0.01 mm
- net +3V3: track 187.0 -> 185.9 mm
- net GND: vias 25 -> 26
