File: WDebug_KiCAD/WDebug_KiCAD/WDebug_KiCAD.sch (KiCad schematic (older format))
At the start: 47 parts, among them J1 USB_C_Receptacle_USB2.0, J2 HD2*10, J3 20p, J4 18p, SW1 sw, U1 USB2514B_Bi, U2 CH340E, U3 CH340E, U4 SPX3819M5-L, Y1 24MHz

Commit message: 修改电阻电容封装
Parts:
- C1, C10, C11, C13, C14, C2, C3, C4, C5, C6, C7, C9: footprint lc_lib:0603_C -> Capacitor_SMD:C_0603_1608Metric
- C12, C8: footprint lc_lib:1206_C -> Capacitor_SMD:C_1206_3216Metric
- D1, D2: footprint digikey-footprints:LED_0603 -> LED_SMD:LED_0603_1608Metric
- R1, R10, R11, R12, R13, R14, R15, R16, R17, R18, R19, R2, R24, R25, R3, R4, R5, R6, R7, R8, R9: footprint lc_lib:0603_R -> Resistor_SMD:R_0603_1608Metric
Changed lines of the file:
@@
 F 0 "C3" V 2850 3850 50  0000 L CNN
 F 1 "100nF" V 2850 3450 50  0000 L CNN
-F 2 "lc_lib:0603_C" H 2838 3600 50  0001 C CNN
+F 2 "Capacitor_SMD:C_0603_1608Metric" H 2838 3600 50  0001 C CNN
 F 3 "~" H 2800 3750 50  0001 C CNN
 	1    2800 3750
@@
 F 0 "R6" V 3150 3400 50  0000 L CNN
 F 1 "12k" V 3150 3100 50  0000 L CNN
-F 2 "lc_lib:0603_R" H 3100 3300 50  0001 C CNN
+F 2 "Resistor_SMD:R_0603_1608Metric" H 3100 3300 50  0001 C CNN
 F 3 "~" H 3100 3300 50  0001 C CNN
 	1    3100 3300
@@
 F 0 "C1" H 1265 5746 50  0000 L CNN
 F 1 "22pF" H 1265 5655 50  0000 L CNN
-F 2 "lc_lib:0603_C" H 1188 5550 50  0001 C CNN
+F 2 "Capacitor_SMD:C_0603_1608Metric" H 1188 5550 50  0001 C CNN
 F 3 "~" H 1150 5700 50  0001 C CNN
 	1    1150 5700
@@
 F 0 "C2" H 2015 5746 50  0000 L CNN
 F 1 "22pF" H 2015 5655 50  0000 L CNN
-F 2 "lc_lib:0603_C" H 1938 5550 50  0001 C CNN
+F 2 "Capacitor_SMD:C_0603_1608Metric" H 1938 5550 50  0001 C CNN
 F 3 "~" H 1900 5700 50  0001 C CNN
 	1    1900 5700
@@
 F 0 "R1" V 1345 4750 50  0000 C CNN
 F 1 "1M" V 1436 4750 50  0000 C CNN
-F 2 "lc_lib:0603_R" H 1550 4750 50  0001 C CNN
+F 2 "Resistor_SMD:R_0603_1608Metric" H 1550 4750 50  0001 C CNN
 F 3 "~" H 1550 4750 50  0001 C CNN
 	1    1550 4750
@@
 F 0 "C4" V 2850 4150 50  0000 L CNN
 F 1 "100nF" V 2850 3750 50  0000 L CNN
-F 2 "lc_lib:0603_C" H 2838 3900 50  0001 C CNN
+F 2 "Capacitor_SMD:C_0603_1608Metric" H 2838 3900 50  0001 C CNN
 F 3 "~" H 2800 4050 50  0001 C CNN
 	1    2800 4050
@@
 F 0 "R2" H 2200 6700 50  0000 L CNN
 F 1 "1K" H 2150 6450 50  0000 L CNN
-F 2 "lc_lib:0603_R" H 2150 6600 50  0001 C CNN
+F 2 "Resistor_SMD:R_0603_1608Metric" H 2150 6600 50  0001 C CNN
 F 3 "~" H 2150 6600 50  0001 C CNN
 	1    2150 6600
@@
 F 0 "R4" H 2600 6700 50  0000 L CNN
 F 1 "1K" H 2550 6450 50  0000 L CNN
-F 2 "lc_lib:0603_R" H 2550 6600 50  0001 C CNN
+F 2 "Resistor_SMD:R_0603_1608Metric" H 2550 6600 50  0001 C CNN
 F 3 "~" H 2550 6600 50  0001 C CNN
 	1    2550 6600
@@
 F 0 "R3" H 2400 6700 50  0000 L CNN
 F 1 "100R" H 2350 6450 50  0000 L CNN
-F 2 "lc_lib:0603_R" H 2350 6600 50  0001 C CNN
+F 2 "Resistor_SMD:R_0603_1608Metric" H 2350 6600 50  0001 C CNN
 F 3 "~" H 2350 6600 50  0001 C CNN
 	1    2350 6600
@@
 F 0 "R5" H 2800 6700 50  0000 L CNN
 F 1 "100R" H 2750 6450 50  0000 L CNN
-F 2 "lc_lib:0603_R" H 2750 6600 50  0001 C CNN
+F 2 "Resistor_SMD:R_0603_1608Metric" H 2750 6600 50  0001 C CNN
 F 3 "~" H 2750 6600 50  0001 C CNN
 	1    2750 6600
@@
 F 0 "R8" H 3518 7196 50  0000 L CNN
 F 1 "10K" H 3518 7105 50  0000 L CNN
-F 2 "lc_lib:0603_R" H 3450 7150 50  0001 C CNN
+F 2 "Resistor_SMD:R_0603_1608Metric" H 3450 7150 50  0001 C CNN
 F 3 "~" H 3450 7150 50  0001 C CNN
 	1    3450 7150
@@
 F 0 "R10" H 3918 7196 50  0000 L CNN
 F 1 "NC" H 3918 7105 50  0000 L CNN
-F 2 "lc_lib:0603_R" H 3850 7150 50  0001 C CNN
+F 2 "Resistor_SMD:R_0603_1608Metric" H 3850 7150 50  0001 C CNN
 F 3 "~" H 3850 7150 50  0001 C CNN
 	1    3850 7150
@@
 F 0 "R7" H 3518 6846 50  0000 L CNN
 F 1 "NC" H 3518 6755 50  0000 L CNN
-F 2 "lc_lib:0603_R" H 3450 6800 50  0001 C CNN
+F 2 "Resistor_SMD:R_0603_1608Metric" H 3450 6800 50  0001 C CNN
 F 3 "~" H 3450 6800 50  0001 C CNN
 	1    3450 6800
@@
 F 0 "D1" V 2389 6933 50  0000 R CNN
 F 1 "GRN" V 2298 6933 50  0000 R CNN
-F 2 "digikey-footprints:LED_0603" H 2350 7050 50  0001 C CNN
+F 2 "LED_SMD:LED_0603_1608Metric" H 2350 7050 50  0001 C CNN
 F 3 "~" H 2350 7050 50  0001 C CNN
 	1    2350 7050
@@
 F 0 "D2" V 2789 6933 50  0000 R CNN
 F 1 "RED" V 2698 6933 50  0000 R CNN
-F 2 "digikey-footprints:LED_0603" H 2750 7050 50  0001 C CNN
+F 2 "LED_SMD:LED_0603_1608Metric" H 2750 7050 50  0001 C CNN
 F 3 "~" H 2750 7050 50  0001 C CNN
 	1    2750 7050
@@
 F 0 "R9" H 3918 6846 50  0000 L CNN
 F 1 "10K" H 3918 6755 50  0000 L CNN
-F 2 "lc_lib:0603_R" H 3850 6800 50  0001 C CNN
+F 2 "Resistor_SMD:R_0603_1608Metric" H 3850 6800 50  0001 C CNN
 F 3 "~" H 3850 6800 50  0001 C CNN
 	1    3850 6800
@@
 F 0 "R11" H 4968 6696 50  0000 L CNN
 F 1 "10K" H 4968 6605 50  0000 L CNN
-F 2 "lc_lib:0603_R" H 4900 6650 50  0001 C CNN
+F 2 "Resistor_SMD:R_0603_1608Metric" H 4900 6650 50  0001 C CNN
 F 3 "~" H 4900 6650 50  0001 C CNN
 	1    4900 6650
@@
 F 0 "C5" H 5015 7246 50  0000 L CNN
 F 1 "1uF" H 5015 7155 50  0000 L CNN
-F 2 "lc_lib:0603_C" H 4938 7050 50  0001 C CNN
+F 2 "Capacitor_SMD:C_0603_1608Metric" H 4938 7050 50  0001 C CNN
 F 3 "~" H 4900 7200 50  0001 C CNN
 	1    4900 7200
@@
 F 0 "C7" H 10365 3146 50  0000 L CNN
 F 1 "0.1uF" H 10365 3055 50  0000 L CNN
-F 2 "lc_lib:0603_C" H 10288 2950 50  0001 C CNN
+F 2 "Capacitor_SMD:C_0603_1608Metric" H 10288 2950 50  0001 C CNN
 F 3 "~" H 10250 3100 50  0001 C CNN
 	1    10250 3100
@@
 F 0 "C6" H 10365 1696 50  0000 L CNN
 F 1 "0.1uF" H 10365 1605 50  0000 L CNN
-F 2 "lc_lib:0603_C" H 10288 1500 50  0001 C CNN
+F 2 "Capacitor_SMD:C_0603_1608Metric" H 10288 1500 50  0001 C CNN
 F 3 "~" H 10250 1650 50  0001 C CNN
 	1    10250 1650
@@
 F 0 "R18" V 10100 2200 50  0000 C CNN
 F 1 "820R" V 10100 1950 50  0000 C CNN
-F 2 "lc_lib:0603_R" H 10150 2100 50  0001 C CNN
+F 2 "Resistor_SMD:R_0603_1608Metric" H 10150 2100 50  0001 C CNN
 F 3 "~" H 10150 2100 50  0001 C CNN
 	1    10150 2100
@@
 F 0 "R19" V 10100 2100 50  0000 C CNN
 F 1 "22R" V 10100 1850 50  0000 C CNN
-F 2 "lc_lib:0603_R" H 10150 2000 50  0001 C CNN
+F 2 "Resistor_SMD:R_0603_1608Metric" H 10150 2000 50  0001 C CNN
 F 3 "~" H 10150 2000 50  0001 C CNN
 	1    10150 2000
@@
 F 0 "R14" V 6200 5100 50  0000 C CNN
 F 1 "10K" V 6200 5350 50  0000 C CNN
-F 2 "lc_lib:0603_R" H 6250 5200 50  0001 C CNN
+F 2 "Resistor_SMD:R_0603_1608Metric" H 6250 5200 50  0001 C CNN
 F 3 "~" H 6250 5200 50  0001 C CNN
 	1    6250 5200
@@
 F 0 "R15" V 6200 5200 50  0000 C CNN
 F 1 "10K" V 6200 5450 50  0000 C CNN
-F 2 "lc_lib:0603_R" H 6250 5300 50  0001 C CNN
+F 2 "Resistor_SMD:R_0603_1608Metric" H 6250 5300 50  0001 C CNN
 F 3 "~" H 6250 5300 50  0001 C CNN
 	1    6250 5300
@@
 F 0 "R12" V 5650 5200 50  0000 C CNN
 F 1 "10K" V 5650 5450 50  0000 C CNN
-F 2 "lc_lib:0603_R" H 5700 5300 50  0001 C CNN
+F 2 "Resistor_SMD:R_0603_1608Metric" H 5700 5300 50  0001 C CNN
 F 3 "~" H 5700 5300 50  0001 C CNN
 	1    5700 5300
@@
 F 0 "R13" V 5750 5400 50  0000 C CNN
 F 1 "10K" V 5750 5600 50  0000 C CNN
-F 2 "lc_lib:0603_R" H 5800 5500 50  0001 C CNN
+F 2 "Resistor_SMD:R_0603_1608Metric" H 5800 5500 50  0001 C CNN
 F 3 "~" H 5800 5500 50  0001 C CNN
 	1    5800 5500
@@
 F 0 "R24" V 5950 6200 50  0000 C CNN
 F 1 "110R" V 5950 6450 50  0000 C CNN
-F 2 "lc_lib:0603_R" H 6000 6300 50  0001 C CNN
+F 2 "Resistor_SMD:R_0603_1608Metric" H 6000 6300 50  0001 C CNN
 F 3 "~" H 6000 6300 50  0001 C CNN
 	1    6000 6300
@@
 F 0 "C9" H 6350 6900 50  0000 L CNN
 F 1 "100nF" H 6350 6600 50  0000 L CNN
-F 2 "lc_lib:0603_C" H 6338 6650 50  0001 C CNN
+F 2 "Capacitor_SMD:C_0603_1608Metric" H 6338 6650 50  0001 C CNN
 F 3 "~" H 6300 6800 50  0001 C CNN
 	1    6300 6800
@@
 F 0 "R25" V 6700 1100 50  0000 C CNN
 F 1 "10K" V 6700 1300 50  0000 C CNN
-F 2 "lc_lib:0603_R" H 6750 1200 50  0001 C CNN
+F 2 "Resistor_SMD:R_0603_1608Metric" H 6750 1200 50  0001 C CNN
 F 3 "~" H 6750 1200 50  0001 C CNN
 	1    6750 1200
@@
 F 0 "C8" H 5950 1650 50  0000 L CNN
 F 1 "10uF" H 5950 1450 50  0000 L CNN
-F 2 "lc_lib:1206_C" H 5938 1400 50  0001 C CNN
+F 2 "Capacitor_SMD:C_1206_3216Metric" H 5938 1400 50  0001 C CNN
 F 3 "~" H 5900 1550 50  0001 C CNN
 	1    5900 1550
@@
 F 0 "C10" H 6250 1650 50  0000 L CNN
 F 1 "100nF" H 6250 1450 50  0000 L CNN
-F 2 "lc_lib:0603_C" H 6238 1400 50  0001 C CNN
+F 2 "Capacitor_SMD:C_0603_1608Metric" H 6238 1400 50  0001 C CNN
 F 3 "~" H 6200 1550 50  0001 C CNN
 	1    6200 1550
@@
 F 0 "C11" H 6550 1650 50  0000 L CNN
 F 1 "220pF" H 6550 1450 50  0000 L CNN
-F 2 "lc_lib:0603_C" H 6538 1400 50  0001 C CNN
+F 2 "Capacitor_SMD:C_0603_1608Metric" H 6538 1400 50  0001 C CNN
 F 3 "~" H 6500 1550 50  0001 C CNN
 	1    6500 1550
@@
 F 0 "C12" H 7750 1650 50  0000 L CNN
 F 1 "10uF" H 7750 1450 50  0000 L CNN
-F 2 "lc_lib:1206_C" H 7738 1400 50  0001 C CNN
+F 2 "Capacitor_SMD:C_1206_3216Metric" H 7738 1400 50  0001 C CNN
 F 3 "~" H 7700 1550 50  0001 C CNN
 	1    7700 1550
@@
 F 0 "C13" H 8050 1650 50  0000 L CNN
 F 1 "100nF" H 8050 1450 50  0000 L CNN
-F 2 "lc_lib:0603_C" H 8038 1400 50  0001 C CNN
+F 2 "Capacitor_SMD:C_0603_1608Metric" H 8038 1400 50  0001 C CNN
 F 3 "~" H 8000 1550 50  0001 C CNN
 	1    8000 1550
@@
 F 0 "C14" H 8350 1650 50  0000 L CNN
 F 1 "100nF" H 8350 1450 50  0000 L CNN
-F 2 "lc_lib:0603_C" H 8338 1400 50  0001 C CNN
+F 2 "Capacitor_SMD:C_0603_1608Metric" H 8338 1400 50  0001 C CNN
 F 3 "~" H 8300 1550 50  0001 C CNN
 	1    8300 1550
@@
 F 0 "R16" V 10150 3600 50  0000 C CNN
 F 1 "820R" V 10150 3350 50  0000 C CNN
-F 2 "lc_lib:0603_R" H 10200 3500 50  0001 C CNN
+F 2 "Resistor_SMD:R_0603_1608Metric" H 10200 3500 50  0001 C CNN
 F 3 "~" H 10200 3500 50  0001 C CNN
 	1    10200 3500
@@
 F 0 "R17" V 10150 3500 50  0000 C CNN
 F 1 "22R" V 10150 3300 50  0000 C CNN
-F 2 "lc_lib:0603_R" H 10200 3400 50  0001 C CNN
+F 2 "Resistor_SMD:R_0603_1608Metric" H 10200 3400 50  0001 C CNN
 F 3 "~" H 10200 3400 50  0001 C CNN
 	1    10200 3400

Commit message: WDebug——DAPLinkV1.2 调整中
Parts:
- SW1: symbol matrix_control_main-cache:matrix_control_main-rescue_switch-LibCool-hack_clock-rescue -> WDebug_KiCAD-rescue:matrix_control_main-rescue_switch-LibCool-hack_clock-rescue-matrix_control_main-cache
- U2, U3: symbol matrix_control_main-cache:matrix_control_main-rescue_CH340E-LibCool-hack_clock-rescue -> WDebug_KiCAD-rescue:matrix_control_main-rescue_CH340E-LibCool-hack_clock-rescue-matrix_control_main-cache
Changed lines of the file:
@@
 EESchema Schematic File Version 4
-LIBS:WDebug_KiCAD-cache
 EELAYER 30 0
 EELAYER END
@@
 $EndDescr
 $Comp
-L matrix_control_main-cache:matrix_control_main-rescue_CH340E-LibCool-hack_clock-rescue U2
+L WDebug_KiCAD-rescue:matrix_control_main-rescue_CH340E-LibCool-hack_clock-rescue-matrix_control_main-cache U2
 U 1 1 5E0A5A6D
 P 9450 2100
@@
 $EndComp
 $Comp
-L matrix_control_main-cache:matrix_control_main-rescue_CH340E-LibCool-hack_clock-rescue U3
+L WDebug_KiCAD-rescue:matrix_control_main-rescue_CH340E-LibCool-hack_clock-rescue-matrix_control_main-cache U3
 U 1 1 5E0A647A
 P 9500 3500
@@
 $EndComp
 $Comp
-L matrix_control_main-cache:matrix_control_main-rescue_switch-LibCool-hack_clock-rescue SW1
+L WDebug_KiCAD-rescue:matrix_control_main-rescue_switch-LibCool-hack_clock-rescue-matrix_control_main-cache SW1
 U 1 1 5E3DE2F5
 P 6600 6800

Commit message: 修正DAPlink 1.5版本 串口信号修改，新加一路串口
Parts:
- C1, C10, C11, C12, C13, C14, C2, C3, C4, C5, C6, C7, C8, C9: symbol Device:C -> WDebug_KiCAD-rescue:C-Device
- D1, D2: symbol Device:LED -> WDebug_KiCAD-rescue:LED-Device
- J1: symbol Connector:USB_C_Receptacle_USB2.0 -> WDebug_KiCAD-rescue:USB_C_Receptacle_USB2.0-Connector
- J2: symbol Connector_Generic:Conn_02x10_Odd_Even -> WDebug_KiCAD-rescue:Conn_02x10_Odd_Even-Connector_Generic
- J3: symbol Connector:Conn_01x20_Female -> WDebug_KiCAD-rescue:Conn_01x20_Female-Connector
- J4: symbol Connector:Conn_01x18_Female -> WDebug_KiCAD-rescue:Conn_01x18_Female-Connector
- R1, R10, R11, R12, R13, R14, R15, R16, R17, R18, R19, R2, R24, R25, R3, R4, R5, R6, R7, R8, R9: symbol Device:R_Small_US -> WDebug_KiCAD-rescue:R_Small_US-Device
- U1: symbol Interface_USB:USB2514B_Bi -> WDebug_KiCAD-rescue:USB2514B_Bi-Interface_USB
- U4: symbol Regulator_Linear:SPX3819M5-L -> WDebug_KiCAD-rescue:SPX3819M5-L-Regulator_Linear
- Y1: symbol Device:Crystal_GND24 -> WDebug_KiCAD-rescue:Crystal_GND24-Device
