File: WDebug_KiCAD/WDebug_DAPLink_KiCAD/WDebug_DAPLink_KiCAD.sch (KiCad schematic (older format))
At the start: 34 parts, among them J1 Conn_01x04, J2 Conn_01x05, J3 Conn_01x05, J4 Conn_02x10_Odd_Even, P1 USB_C_Plug_USB2.0, U1 AZ1117-3.3, U2 STM32F103C8Tx, Y1 8MHz

Commit message: 第二版可以正常烧写，有串口
Parts:
- removed J2, J3: Conn_01x05, Connector_Harwin:Harwin_M20-89005xx_1x05_P2.54mm_Horizontal, symbol Connector_Generic:Conn_01x05
- removed J4: Conn_02x10_Odd_Even, Connector_PinHeader_2.54mm:PinHeader_2x10_P2.54mm_Vertical, symbol Connector_Generic:Conn_02x10_Odd_Even
- added C11: 100nF, Capacitor_SMD:C_0603_1608Metric, symbol Device:C
- added J2: Conn_02x04_UART_SW, Connector_PinSocket_2.54mm:PinSocket_2x04_P2.54mm_Vertical, symbol Connector_Generic:Conn_02x04_Top_Bottom
- added J5: Conn_01x18_Female, WDebug_KiCAD:1x16_P1.0mm, symbol Connector:Conn_01x18_Female
- added R14: 10k, Resistor_SMD:R_0603_1608Metric, symbol Device:R_Small_US
- added R15: 100R, Resistor_SMD:R_0603_1608Metric, symbol Device:R_Small_US
- added SW1: SW_Rst, matrix_control_main:SWITCH_PUSH, symbol Switch:SW_Push
- C1: footprint Capacitor_SMD:C_1206_3216Metric -> Capacitor_SMD:C_0603_1608Metric
- R10, R8: value 100K -> 10K
- U2: symbol DAPLink-cache:MCU_ST_STM32F1_STM32F103C8Tx -> WDebug_DAPLink_KiCAD-rescue:MCU_ST_STM32F1_STM32F103C8Tx-DAPLink-cache
Connections:
- net labels added: RX1, RX2, TX1, TX2
- net labels removed: USB3+, USB3-
- wire segments 188 -> 177
- no-connect marks 25 -> 26

Commit message: WDebug——DAPLinkV1.2 调整中
Parts:
- removed R9: 100R, Resistor_SMD:R_0603_1608Metric, symbol Device:R_Small_US
- added J3: Conn_01x20_Female, WDebug_KiCAD:1x18_P1.0mm, symbol Connector:Conn_01x20_Female
- added J4: Conn_01x05_Male, Connector_PinHeader_2.54mm:PinHeader_1x05_P2.54mm_Vertical, symbol Connector:Conn_01x05_Male
- J2: footprint Connector_PinSocket_2.54mm:PinSocket_2x04_P2.54mm_Vertical -> Connector_PinHeader_2.54mm:PinHeader_2x04_P2.54mm_Vertical
- U2: symbol WDebug_DAPLink_KiCAD-rescue:MCU_ST_STM32F1_STM32F103C8Tx-DAPLink-cache -> WDebug_DAPLink_KiCAD-rescue:MCU_ST_STM32F1_STM32F103C8Tx-DAPLink-cache-WDebug_DAPLink_KiCAD-rescue
- Y1: footprint Crystal:Crystal_SMD_5032-4Pin_5.0x3.2mm -> Crystal:Crystal_SMD_3225-4Pin_3.2x2.5mm
Connections:
- wire segments 177 -> 180
- no-connect marks 26 -> 27

Commit message: 修改好DAPLinkV1.2版本
Parts:
- C1, C10, C11, C2, C3, C4, C5, C7, C8, C9: symbol Device:C -> WDebug_DAPLink_KiCAD-rescue:C-Device
- C6: footprint Capacitor_SMD:C_1206_3216Metric -> Capacitor_SMD:C_0603_1608Metric; symbol Device:C -> WDebug_DAPLink_KiCAD-rescue:C-Device
- D1, D2, D3: symbol Device:LED -> WDebug_DAPLink_KiCAD-rescue:LED-Device
- J1: symbol Connector_Generic:Conn_01x04 -> WDebug_DAPLink_KiCAD-rescue:Conn_01x04-Connector_Generic
- J2: symbol Connector_Generic:Conn_02x04_Top_Bottom -> WDebug_DAPLink_KiCAD-rescue:Conn_02x04_Top_Bottom-Connector_Generic
- J5: value Conn_01x18_Female -> 01x18_Female_Fan
- R1, R10, R11, R12, R13, R14, R15, R2, R3, R4, R5, R6, R7, R8: symbol Device:R_Small_US -> WDebug_DAPLink_KiCAD-rescue:R_Small_US-Device
- SW1: symbol Switch:SW_Push -> WDebug_DAPLink_KiCAD-rescue:SW_Push-Switch
- U1: symbol Regulator_Linear:AZ1117-3.3 -> WDebug_DAPLink_KiCAD-rescue:AZ1117-3.3-Regulator_Linear
- U2: symbol WDebug_DAPLink_KiCAD-rescue:MCU_ST_STM32F1_STM32F103C8Tx-DAPLink-cache-WDebug_DAPLink_KiCAD-rescue -> WDebug_DAPLink_KiCAD-rescue:MCU_ST_STM32F1_STM32F103C8Tx-DAPLink-cache-WDebug_DAPLink_KiCAD-rescue-WDebug_DAPLink_KiCAD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
- Y1: symbol Device:Crystal_GND24 -> WDebug_DAPLink_KiCAD-rescue:Crystal_GND24-Device
Connections:
- wire segments 180 -> 196
- no-connect marks 27 -> 35

Commit message: 提交修改USB type-C和按键 3D模型
Parts:
- P1: footprint matrix_control_main:USB-Type-C -> WDebug_DAPLink:USB-Type-C
- SW1: footprint matrix_control_main:SWITCH_PUSH -> WDebug_DAPLink:SWITCH_PUSH
Changed lines of the file:
@@
 F 0 "P1" H 1807 3217 50  0000 C CNN
 F 1 "USB_C_Plug_USB2.0" H 1807 3126 50  0000 C CNN
-F 2 "matrix_control_main:USB-Type-C" H 1850 2350 50  0001 C CNN
+F 2 "WDebug_DAPLink:USB-Type-C" H 1850 2350 50  0001 C CNN
 F 3 "https://www.usb.org/sites/default/files/documents/usb_type-c.zip" H 1850 2350 50  0001 C CNN
 	1    1700 2350
@@
 F 0 "SW1" V 10404 5848 50  0000 L CNN
 F 1 "SW_Rst" V 10495 5848 50  0000 L CNN
-F 2 "matrix_control_main:SWITCH_PUSH" H 10450 5900 50  0001 C CNN
+F 2 "WDebug_DAPLink:SWITCH_PUSH" H 10450 5900 50  0001 C CNN
 F 3 "~" H 10450 5900 50  0001 C CNN
 	1    10450 5700
@@
 T_SWO
 $Comp
-L WDebug_DAPLink_KiCAD-rescue:+3.3V-power #PWR?
+L WDebug_DAPLink_KiCAD-rescue:+3.3V-power #PWR0124
 U 1 1 5EA83DB7
 P 4950 6000
-F 0 "#PWR?" H 4950 5850 50  0001 C CNN
+F 0 "#PWR0124" H 4950 5850 50  0001 C CNN
 F 1 "+3.3V" H 4965 6173 50  0000 C CNN
 F 2 "" H 4950 6000 50  0001 C CNN

Commit message: WDebug_KiCAD_V1.3 修改串口RX和TX相反，16pin接口定义相反
Parts:
- J3: symbol Connector:Conn_01x20_Female -> WDebug_DAPLink_KiCAD-rescue:Conn_01x20_Female-Connector
- J4: symbol Connector:Conn_01x05_Male -> WDebug_DAPLink_KiCAD-rescue:Conn_01x05_Male-Connector
- J5: footprint WDebug_KiCAD:1x16_P1.0mm -> WDebug_DAPLink:1x16_P1.0mm; symbol Connector:Conn_01x18_Female -> WDebug_DAPLink_KiCAD-rescue:Conn_01x18_Female-Connector
- P1: symbol Connector:USB_C_Plug_USB2.0 -> WDebug_DAPLink_KiCAD-rescue:USB_C_Plug_USB2.0-Connector
Changed lines of the file:
@@
 $EndComp
 $Comp
-L Connector:USB_C_Plug_USB2.0 P1
+L WDebug_DAPLink_KiCAD-rescue:USB_C_Plug_USB2.0-Connector P1
 U 1 1 5E0DCA6A
 P 1700 2350
@@
 T_TX
 Text Label 5350 3200 0    50   ~ 0
+RX1
+Text Label 5350 3300 0    50   ~ 0
 TX1
-Text Label 5350 3300 0    50   ~ 0
-RX1
 Text Label 5350 3600 0    50   Italic 0
+RX2
+Text Label 5350 3700 0    50   Italic 0
 TX2
-Text Label 5350 3700 0    50   Italic 0
-RX2
 Text Label 5350 3400 0    50   Italic 0
 T_SWCLK
@@
 NoConn ~ 5950 4300
 $Comp
-L Connector:Conn_01x18_Female J5
+L WDebug_DAPLink_KiCAD-rescue:Conn_01x18_Female-Connector J5
 U 1 1 5E948B21
 P 6150 3600
 F 0 "J5" H 6178 3576 50  0000 L CNN
 F 1 "01x18_Female_Fan" H 5800 2550 50  0000 L CNN
-F 2 "WDebug_KiCAD:1x16_P1.0mm" H 6150 3600 50  0001 C CNN
+F 2 "WDebug_DAPLink:1x16_P1.0mm" H 6150 3600 50  0001 C CNN
 F 3 "~" H 6150 3600 50  0001 C CNN
 	1    6150 3600
@@
 TG_RST
 $Comp
-L Connector:Conn_01x20_Female J3
+L WDebug_DAPLink_KiCAD-rescue:Conn_01x20_Female-Connector J3
 U 1 1 5E98C7BB
 P 6150 6250
@@
 NoConn ~ 9600 3450
 $Comp
-L Connector:Conn_01x05_Male J4
+L WDebug_DAPLink_KiCAD-rescue:Conn_01x05_Male-Connector J4
 U 1 1 5E944D28
 P 2350 6800
@@
 	5950 6350 5350 6350
 Text Label 5350 7050 0    50   ~ 0
+TX1
+Text Label 5350 6950 0    50   ~ 0
 RX1
-Text Label 5350 6950 0    50   ~ 0
-TX1
 Text Label 5350 6850 0    50   ~ 0
 T_SWCLK
@@
 TG_RST
 Text Label 5350 6250 0    50   ~ 0
+TX2
+Text Label 5350 6150 0    50   ~ 0
 RX2
-Text Label 5350 6150 0    50   ~ 0
-TX2
 NoConn ~ 5950 5350
 NoConn ~ 5950 5450
