File: WDebug_KiCAD/WDebug_DAPLink_KiCAD/WDebug_DAPLink_KiCAD.sch (KiCad schematic (older format))
At the start: 40 parts, among them J1 Conn_01x04, J2 Conn_02x04_UART_SW, J3 Conn_01x20_Female, J4 Conn_01x05_Male, J5 01x18_Female_Fan, J6 3.3V_Conn, P1 USB_C_Plug_USB2.0, SW1 SW_Rst, U1 XC6228D332VR-G-matrix_display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, U2 STM32F103C8Tx, Y1 8MHz

Commit message: 新加转接板，准备V1.7版本的修改思路和改进点
Parts:
- removed J2: Conn_02x04_UART_SW, Connector_PinHeader_2.54mm:PinHeader_2x04_P2.54mm_Vertical, symbol WDebug_DAPLink_KiCAD-rescue:Conn_02x04_Top_Bottom-Connector_Generic
- removed J3: Conn_01x20_Female, WDebug_KiCAD:1x18_P1.0mm, symbol WDebug_DAPLink_KiCAD-rescue:Conn_01x20_Female-Connector
- removed J4: Conn_01x05_Male, Connector_PinHeader_2.54mm:PinHeader_1x05_P2.54mm_Vertical, symbol WDebug_DAPLink_KiCAD-rescue:Conn_01x05_Male-Connector
- removed J5: 01x18_Female_Fan, WDebug_DAPLink:1x16_P1.0mm, symbol WDebug_DAPLink_KiCAD-rescue:Conn_01x18_Female-Connector
- added J2: ConnDebug, Connector_PinHeader_2.54mm:PinHeader_2x05_P2.54mm_Vertical, symbol WDebug_DAPLink_KiCAD-rescue:Conn_02x05_Counter_Clockwise-Connector_Generic
- C1, C6: footprint Capacitor_SMD:C_0603_1608Metric -> Capacitor_SMD:C_0805_2012Metric
- J6: symbol Connector:Conn_01x02_Female -> WDebug_DAPLink_KiCAD-rescue:Conn_01x02_Female-Connector
- U1: symbol matrix_control_main-rescue:XC6228D332VR-G-matrix_display-rescue -> WDebug_DAPLink_KiCAD-rescue:XC6228D332VR-G-matrix_display-rescue-matrix_control_main-rescue
Connections:
- net +3V3: now also J2.10 (Pin_10); no longer J1.4 (Pin_4)
- net GND: now also J2.5 (Pin_5), J2.6 (Pin_6)
- net IF_RST: now also J1.4 (Pin_4)
- net MCU_RX1: now also J2.1 (Pin_1)
- net MCU_RX2: now also J2.2 (Pin_2)
- net MCU_TX1: now also J2.3 (Pin_3)
- net MCU_TX2: now also J2.4 (Pin_4)
- net TG_RST: now also J2.7 (Pin_7)
- net T_SWCLK: now also J2.9 (Pin_9)
- net T_SWDIO: now also J2.8 (Pin_8)
- no-connect marks 35 -> 21
Other:
- moved on the sheet: J6
