File: matrix_display16_32/matrix_display16_32.sch (KiCad schematic (older format))
At the start: 29 parts, among them J1 Conn_01x05_Male, U1 MAX7219, U10 Matrix_LED, U11 Matrix_LED, U12 Matrix_LED, U13 Matrix_LED, U14 Matrix_LED, U15 Matrix_LED, U16 Matrix_LED, U2 MAX7219, U3 MAX7219, U4 MAX7219, U5 MAX7219, U6 MAX7219, U7 MAX7219, U8 MAX7219, U9 Matrix_LED

Commit message: 修改点阵铜柱洞3.5MM 修改连接接口2.54MM
Parts:
- C1, C2, C3, C4: symbol matrix_display-rescue:C(MM)-LibCool -> matrix_display16_32-rescue:C(MM)-LibCool-matrix_display-rescue
- J1: footprint Connector_PinHeader_2.00mm:PinHeader_1x05_P2.00mm_Vertical -> Connector_PinHeader_2.54mm:PinHeader_1x05_P2.54mm_Vertical
- R1, R2, R3, R4, R5, R6, R7, R8: symbol matrix_display-rescue:RES(M)-LibCool -> matrix_display16_32-rescue:RES(M)-LibCool-matrix_display-rescue
- U1, U2, U3, U4, U5, U6, U7, U8: symbol Driver_LED:MAX7219 -> matrix_display16_32-rescue:MAX7219-Driver_LED
- U10, U11, U12, U13, U14, U15, U16, U9: symbol matrix_display-rescue:Matrix_LED-LibCool -> matrix_display16_32-rescue:Matrix_LED-LibCool-matrix_display-rescue
Changed lines of the file:
@@
 EESchema Schematic File Version 4
-LIBS:matrix_display16_32-cache
 EELAYER 30 0
 EELAYER END
@@
 F 0 "J1" H 4708 9781 50  0000 C CNN
 F 1 "Conn_01x05_Male" H 4708 9690 50  0000 C CNN
-F 2 "Connector_PinHeader_2.00mm:PinHeader_1x05_P2.00mm_Vertical" H 4600 9400 50  0001 C CNN
+F 2 "Connector_PinHeader_2.54mm:PinHeader_1x05_P2.54mm_Vertical" H 4600 9400 50  0001 C CNN
 F 3 "~" H 4600 9400 50  0001 C CNN
 	1    4600 9400
@@
 	10150 4250 10000 4250
 $Comp
-L matrix_display-rescue:Matrix_LED-LibCool U11
+L matrix_display16_32-rescue:Matrix_LED-LibCool-matrix_display-rescue U11
 U 1 1 5DD4E45D
 P 11050 4200
@@
 CS
 $Comp
-L matrix_display-rescue:RES(M)-LibCool R6
+L matrix_display16_32-rescue:RES(M)-LibCool-matrix_display-rescue R6
 U 1 1 5DD62A59
 P 3550 5750
@@
 	3550 5900 3650 5900
 $Comp
-L matrix_display-rescue:Matrix_LED-LibCool U9
+L matrix_display16_32-rescue:Matrix_LED-LibCool-matrix_display-rescue U9
 U 1 1 5DD05F05
 P 11000 2550
@@
 1_DIG0
 $Comp
-L matrix_display-rescue:Matrix_LED-LibCool U12
+L matrix_display16_32-rescue:Matrix_LED-LibCool-matrix_display-rescue U12
 U 1 1 5DD62AA4
 P 13250 4200
@@
 	4050 5500 4050 5600
 $Comp
-L Driver_LED:MAX7219 U6
+L matrix_display16_32-rescue:MAX7219-Driver_LED U6
 U 1 1 5DD62A4D
 P 4050 6700
@@
 $EndComp
 $Comp
-L matrix_display-rescue:Matrix_LED-LibCool U10
+L matrix_display16_32-rescue:Matrix_LED-LibCool-matrix_display-rescue U10
 U 1 1 5DD56516
 P 13250 2550
@@
 	2500 5500 2500 5600
 $Comp
-L matrix_display-rescue:RES(M)-LibCool R5
+L matrix_display16_32-rescue:RES(M)-LibCool-matrix_display-rescue R5
 U 1 1 5DD4E412
 P 2000 5750
@@
 	2100 7400 1750 7400
 $Comp
-L Driver_LED:MAX7219 U5
+L matrix_display16_32-rescue:MAX7219-Driver_LED U5
 U 1 1 5DD4E406
 P 2500 6700
@@
 CS
 $Comp
-L matrix_display-rescue:RES(M)-LibCool R8
+L matrix_display16_32-rescue:RES(M)-LibCool-matrix_display-rescue R8
 U 1 1 5DEF73BA
 P 6700 5750
@@
 	7200 5500 7200 5600
 $Comp
-L Driver_LED:MAX7219 U8
+L matrix_display16_32-rescue:MAX7219-Driver_LED U8
 U 1 1 5DEF73F0
 P 7200 6700
@@
 	5650 5500 5650 5600
 $Comp
-L matrix_display-rescue:RES(M)-LibCool R7
+L matrix_display16_32-rescue:RES(M)-LibCool-matrix_display-rescue R7
 U 1 1 5DEF745E
 P 5150 5750
@@
 	5250 7400 4900 7400
 $Comp
-L Driver_LED:MAX7219 U7
+L matrix_display16_32-rescue:MAX7219-Driver_LED U7
 U 1 1 5DEF746A
 P 5650 6700
@@
 	10200 7750 10050 7750
 $Comp
-L matrix_display-rescue:Matrix_LED-LibCool U15
+L matrix_display16_32-rescue:Matrix_LED-LibCool-matrix_display-rescue U15
 U 1 1 5DF970C6
 P 11100 7700
@@
 $EndComp
 $Comp
-L matrix_display-rescue:Matrix_LED-LibCool U13
+L matrix_display16_32-rescue:Matrix_LED-LibCool-matrix_display-rescue U13
 U 1 1 5DF970CC
 P 11050 6050
@@
 5_DIG7
 $Comp
-L matrix_display-rescue:Matrix_LED-LibCool U16
+L matrix_display16_32-rescue:Matrix_LED-LibCool-matrix_display-rescue U16
 U 1 1 5DF970E2
 P 13300 7700
@@
 8_SEGA
 $Comp
-L matrix_display-rescue:Matrix_LED-LibCool U14
+L matrix_display16_32-rescue:Matrix_LED-LibCool-matrix_display-rescue U14
 U 1 1 5DF97108
 P 13300 6050
@@
 	2900 4450 3650 4450
 $Comp
-L Driver_LED:MAX7219 U4
+L matrix_display16_32-rescue:MAX7219-Driver_LED U4
 U 1 1 5DEF7420
 P 7200 3650
@@
 	6700 2550 7200 2550
 $Comp
-L Driver_LED:MAX7219 U3
+L matrix_display16_32-rescue:MAX7219-Driver_LED U3
 U 1 1 5DEF73C6
 P 5650 3650
@@
 	6700 2850 6800 2850
 $Comp
-L matrix_display-rescue:RES(M)-LibCool R4
+L matrix_display16_32-rescue:RES(M)-LibCool-matrix_display-rescue R4
 U 1 1 5DEF73A6
 P 6700 2700
@@
 	5650 2450 5650 2550
 $Comp
-L matrix_display-rescue:RES(M)-LibCool R3
+L matrix_display16_32-rescue:RES(M)-LibCool-matrix_display-rescue R3
 U 1 1 5DEF7377
 P 5150 2700
@@
 	4050 4850 4050 4650
 $Comp
-L Driver_LED:MAX7219 U2
+L matrix_display16_32-rescue:MAX7219-Driver_LED U2
 U 1 1 5DD564BF
 P 4050 3650
@@
 2_DIG7
 $Comp
-L Driver_LED:MAX7219 U1
+L matrix_display16_32-rescue:MAX7219-Driver_LED U1
 U 1 1 5DCF699B
 P 2500 3650
@@
 	3550 2850 3650 2850
 $Comp
-L matrix_display-rescue:RES(M)-LibCool R2
+L matrix_display16_32-rescue:RES(M)-LibCool-matrix_display-rescue R2
 U 1 1 5DD564CB
 P 3550 2700
@@
 	2500 2450 2500 2550
 $Comp
-L matrix_display-rescue:RES(M)-LibCool R1
+L matrix_display16_32-rescue:RES(M)-LibCool-matrix_display-rescue R1
 U 1 1 5DD0F649
 P 2000 2700
@@
 NoConn ~ 14050 7450
 $Comp
-L matrix_display-rescue:C(MM)-LibCool C1
+L matrix_display16_32-rescue:C(MM)-LibCool-matrix_display-rescue C1
 U 1 1 5DE42788
 P 6100 9100
@@
 $EndComp
 $Comp
-L matrix_display-rescue:C(MM)-LibCool C2
+L matrix_display16_32-rescue:C(MM)-LibCool-matrix_display-rescue C2
 U 1 1 5DE70AC3
 P 6350 9100
@@
 $EndComp
 $Comp
-L matrix_display-rescue:C(MM)-LibCool C3
+L matrix_display16_32-rescue:C(MM)-LibCool-matrix_display-rescue C3
 U 1 1 5DE9A258
 P 6600 9100
@@
 $EndComp
 $Comp
-L matrix_display-rescue:C(MM)-LibCool C4
+L matrix_display16_32-rescue:C(MM)-LibCool-matrix_display-rescue C4
 U 1 1 5DF61206
 P 6850 9100
